File: max33xxE_breakout.sch (EAGLE design)
At the start: 24 parts

Commit message: join the separate VCC and VL segments with solderpads
Parts:
- added SJ1, SJ2, SJ3, SJ4, SJ5, SJ6: SOLDERJUMPERTRACE, SparkFun-Passives:SOLDERJUMPERTRACE
Connections:
- net VCC_SHIFT1: now also SJ1.1
- net VCC_SHIFT2: now also SJ1.2, SJ5.1
- net VCC_SHIFT3: now also SJ4.1, SJ5.2
- net VCC_SHIFT4: now also SJ4.2
- net VL_SHIFT1: now also SJ6.1
- net VL_SHIFT2: now also SJ2.1, SJ6.2
- net VL_SHIFT3: now also SJ2.2, SJ3.1
- net VL_SHIFT4: now also SJ3.2
Changed lines of the file:
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@@
 <layer number="111" name="MPL" color="7" fill="1" visible="yes" active="yes"/>
 <layer number="112" name="tSilk" color="7" fill="1" visible="yes" active="yes"/>
+<layer number="116" name="Patch_BOT" color="9" fill="4" visible="no" active="yes"/>
 <layer number="121" name="sName" color="7" fill="1" visible="yes" active="yes"/>
 <layer number="122" name="_bPlace" color="7" fill="1" visible="yes" active="yes"/>
@@
 <layer number="204" name="204bmp" color="7" fill="1" visible="yes" active="yes"/>
 <layer number="205" name="205bmp" color="7" fill="1" visible="yes" active="yes"/>
+<layer number="206" name="206bmp" color="7" fill="10" visible="no" active="yes"/>
+<layer number="207" name="207bmp" color="8" fill="10" visible="no" active="yes"/>
+<layer number="208" name="208bmp" color="9" fill="10" visible="no" active="yes"/>
+<layer number="209" name="209bmp" color="7" fill="1" visible="no" active="yes"/>
+<layer number="210" name="210bmp" color="7" fill="1" visible="no" active="yes"/>
+<layer number="211" name="211bmp" color="7" fill="1" visible="no" active="yes"/>
+<layer number="212" name="212bmp" color="7" fill="1" visible="no" active="yes"/>
+<layer number="213" name="213bmp" color="7" fill="1" visible="no" active="yes"/>
+<layer number="214" name="214bmp" color="7" fill="1" visible="no" active="yes"/>
+<layer number="215" name="215bmp" color="7" fill="1" visible="no" active="yes"/>
+<layer number="216" name="216bmp" color="7" fill="1" visible="no" active="yes"/>
+<layer number="217" name="217bmp" color="18" fill="1" visible="no" active="no"/>
+<layer number="218" name="218bmp" color="19" fill="1" visible="no" active="no"/>
+<layer number="219" name="219bmp" color="20" fill="1" visible="no" active="no"/>
+<layer number="220" name="220bmp" color="21" fill="1" visible="no" active="no"/>
+<layer number="221" name="221bmp" color="22" fill="1" visible="no" active="no"/>
+<layer number="222" name="222bmp" color="23" fill="1" visible="no" active="no"/>
+<layer number="223" name="223bmp" color="24" fill="1" visible="no" active="no"/>
+<layer number="224" name="224bmp" color="25" fill="1" visible="no" active="no"/>
 <layer number="248" name="Housing" color="7" fill="1" visible="yes" active="yes"/>
 <layer number="249" name="Edge" color="7" fill="1" visible="yes" active="yes"/>
@@
 <part name="GND11" library="supply1" deviceset="GND" device=""/>
 <part name="GND12" library="supply1" deviceset="GND" device=""/>
+<part name="SJ1" library="SparkFun-Passives" deviceset="SOLDERJUMPER" device="TRACE"/>
+<part name="SJ2" library="SparkFun-Passives" deviceset="SOLDERJUMPER" device="TRACE"/>
+<part name="SJ3" library="SparkFun-Passives" deviceset="SOLDERJUMPER" device="TRACE"/>
+<part name="SJ4" library="SparkFun-Passives" deviceset="SOLDERJUMPER" device="TRACE"/>
+<part name="SJ5" library="SparkFun-Passives" deviceset="SOLDERJUMPER" device="TRACE"/>
+<part name="SJ6" library="SparkFun-Passives" deviceset="SOLDERJUMPER" device="TRACE"/>
 </parts>
 <sheets>
@@
 <instance part="GND11" gate="1" x="25.4" y="73.66"/>
 <instance part="GND12" gate="1" x="38.1" y="73.66"/>
+<instance part="SJ1" gate="1" x="83.82" y="88.9"/>
+<instance part="SJ2" gate="1" x="185.42" y="99.06"/>
+<instance part="SJ3" gate="1" x="287.02" y="99.06"/>
+<instance part="SJ4" gate="1" x="287.02" y="106.68"/>
+<instance part="SJ5" gate="1" x="185.42" y="106.68"/>
+<instance part="SJ6" gate="1" x="83.82" y="96.52"/>
 </instances>
 <busses>
@@
 <label x="35.56" y="86.36" size="1.778" layer="95" rot="R90"/>
 </segment>
+<segment>
+<pinref part="SJ1" gate="1" pin="1"/>
+<wire x1="78.74" y1="88.9" x2="71.12" y2="88.9" width="0.1524" layer="91"/>
+<label x="60.96" y="88.9" size="1.778" layer="95"/>
+</segment>
 </net>
 <net name="VL_SHIFT1" class="0">
@@
 <wire x1="25.4" y1="83.82" x2="25.4" y2="88.9" width="0.1524" layer="91"/>
 <label x="22.86" y="86.36" size="1.778" layer="95" rot="R90"/>
+</segment>
+<segment>
+<pinref part="SJ6" gate="1" pin="1"/>
+<wire x1="78.74" y1="96.52" x2="71.12" y2="96.52" width="0.1524" layer="91"/>
+<label x="60.96" y="96.52" size="1.778" layer="95"/>
 </segment>
 </net>
@@
 <label x="124.46" y="101.6" size="1.778" layer="95" rot="R90"/>
 </segment>
+<segment>
+<pinref part="SJ6" gate="1" pin="2"/>
+<wire x1="88.9" y1="96.52" x2="96.52" y2="96.52" width="0.1524" layer="91"/>
+<label x="93.98" y="96.52" size="1.778" layer="95"/>
+</segment>
+<segment>
+<pinref part="SJ2" gate="1" pin="1"/>
+<wire x1="180.34" y1="99.06" x2="172.72" y2="99.06" width="0.1524" layer="91"/>
+<label x="162.56" y="99.06" size="1.778" layer="95"/>
+</segment>
 </net>
 <net name="VCC_SHIFT2" class="0">
@@
 <wire x1="137.16" y1="99.06" x2="137.16" y2="104.14" width="0.1524" layer="91"/>
 <label x="134.62" y="101.6" size="1.778" layer="95" rot="R90"/>
+</segment>
+<segment>
+<pinref part="SJ1" gate="1" pin="2"/>
+<wire x1="88.9" y1="88.9" x2="96.52" y2="88.9" width="0.1524" layer="91"/>
+<label x="93.98" y="88.9" size="1.778" layer="95"/>
+</segment>
+<segment>
+<pinref part="SJ5" gate="1" pin="1"/>
+<wire x1="180.34" y1="106.68" x2="172.72" y2="106.68" width="0.1524" layer="91"/>
+<label x="160.02" y="106.68" size="1.778" layer="95"/>
 </segment>
 </net>
@@
 <label x="220.98" y="104.14" size="1.778" layer="95" rot="R90"/>
 </segment>
+<segment>
+<pinref part="SJ3" gate="1" pin="1"/>
+<wire x1="281.94" y1="99.06" x2="274.32" y2="99.06" width="0.1524" layer="91"/>
+<label x="266.7" y="99.06" size="1.778" layer="95"/>
+</segment>
+<segment>
+<pinref part="SJ2" gate="1" pin="2"/>
+<wire x1="190.5" y1="99.06" x2="198.12" y2="99.06" width="0.1524" layer="91"/>
+<label x="195.58" y="99.06" size="1.778" layer="95"/>
+</segment>
 </net>
 <net name="VCC_SHIFT3" class="0">
@@
 <wire x1="238.76" y1="99.06" x2="238.76" y2="104.14" width="0.1524" layer="91"/>
 <label x="236.22" y="104.14" size="1.778" layer="95" rot="R90"/>
+</segment>
+<segment>
+<pinref part="SJ4" gate="1" pin="1"/>
+<wire x1="281.94" y1="106.68" x2="274.32" y2="106.68" width="0.1524" layer="91"/>
+<label x="264.16" y="106.68" size="1.778" layer="95"/>
+</segment>
+<segment>
+<pinref part="SJ5" gate="1" pin="2"/>
+<wire x1="190.5" y1="106.68" x2="198.12" y2="106.68" width="0.1524" layer="91"/>
+<label x="195.58" y="106.68" size="1.778" layer="95"/>
 </segment>
 </net>
@@
 <label x="317.5" y="106.68" size="1.778" layer="95" rot="R90"/>
 </segment>
+<segment>
+<pinref part="SJ3" gate="1" pin="2"/>
+<wire x1="292.1" y1="99.06" x2="299.72" y2="99.06" width="0.1524" layer="91"/>
+<label x="297.18" y="99.06" size="1.778" layer="95"/>
+</segment>
 </net>
 <net name="VCC_SHIFT4" class="0">
@@
 <label x="332.74" y="106.68" size="1.778" layer="95" rot="R90"/>
 </segment>
-</net>
+<segment>
+<pinref part="SJ4" gate="1" pin="2"/>
+<wire x1="292.1" y1="106.68" x2="299.72" y2="106.68" width="0.1524" layer="91"/>
+<label x="297.18" y="106.68" size="1.778" layer="95"/>
+</segment>
+</net>

Commit message: forgot that the -THREESTATE *must* be pulled to VCC/VL
Connections:
- net VCC_SHIFT1: now also SHIFT1.-3STATE
- net VCC_SHIFT2: now also SHIFT2.-3STATE
- net VCC_SHIFT3: now also SHIFT3.-3STATE
- net VCC_SHIFT4: now also SHIFT4.-3STATE
Changed lines of the file:
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@@
 <pinref part="P+1" gate="1" pin="+5V"/>
 <wire x1="35.56" y1="63.5" x2="35.56" y2="60.96" width="0.1524" layer="91"/>
+<pinref part="SHIFT1" gate="G$1" pin="-3STATE"/>
+<wire x1="17.78" y1="50.8" x2="15.24" y2="50.8" width="0.1524" layer="91"/>
+<wire x1="15.24" y1="50.8" x2="15.24" y2="68.58" width="0.1524" layer="91"/>
+<wire x1="15.24" y1="68.58" x2="40.64" y2="68.58" width="0.1524" layer="91"/>
+<wire x1="40.64" y1="68.58" x2="40.64" y2="60.96" width="0.1524" layer="91"/>
+<wire x1="40.64" y1="60.96" x2="35.56" y2="60.96" width="0.1524" layer="91"/>
+<junction x="35.56" y="60.96"/>
 </segment>
 <segment>
@@
 <wire x1="137.16" y1="60.96" x2="132.08" y2="60.96" width="0.1524" layer="91"/>
 <junction x="132.08" y="60.96"/>
+<pinref part="SHIFT2" gate="G$1" pin="-3STATE"/>
+<wire x1="114.3" y1="50.8" x2="114.3" y2="73.66" width="0.1524" layer="91"/>
+<wire x1="114.3" y1="73.66" x2="137.16" y2="73.66" width="0.1524" layer="91"/>
+<wire x1="137.16" y1="73.66" x2="137.16" y2="66.04" width="0.1524" layer="91"/>
+<junction x="137.16" y="66.04"/>
 </segment>
 <segment>
@@
 <wire x1="233.68" y1="55.88" x2="228.6" y2="55.88" width="0.1524" layer="91"/>
 <junction x="228.6" y="55.88"/>
+<pinref part="SHIFT3" gate="G$1" pin="-3STATE"/>
+<wire x1="210.82" y1="45.72" x2="210.82" y2="68.58" width="0.1524" layer="91"/>
+<wire x1="210.82" y1="68.58" x2="233.68" y2="68.58" width="0.1524" layer="91"/>
+<wire x1="233.68" y1="68.58" x2="233.68" y2="60.96" width="0.1524" layer="91"/>
+<junction x="233.68" y="60.96"/>
 </segment>
 <segment>
@@
 <wire x1="332.74" y1="60.96" x2="327.66" y2="60.96" width="0.1524" layer="91"/>
 <junction x="327.66" y="60.96"/>
-</segment>
-<segment>
+<pinref part="SHIFT4" gate="G$1" pin="-3STATE"/>
+<wire x1="309.88" y1="50.8" x2="309.88" y2="73.66" width="0.1524" layer="91"/>
+<wire x1="309.88" y1="73.66" x2="332.74" y2="73.66" width="0.1524" layer="91"/>
+<wire x1="332.74" y1="73.66" x2="332.74" y2="66.04" width="0.1524" layer="91"/>
+<junction x="332.74" y="66.04"/>
+</segment>
+<segment>

Commit message: daym, -threestate must be pulled VL not VCC, good that I verified this...
Connections:
- new net +5V: SHIFT1.VCC
- net VCC_SHIFT1: no longer SHIFT1.-3STATE, SHIFT1.VCC
- net VCC_SHIFT2: no longer SHIFT2.-3STATE
- net VCC_SHIFT3: no longer SHIFT3.-3STATE
- net VCC_SHIFT4: no longer SHIFT4.-3STATE
- net VL_SHIFT1: now also SHIFT1.-3STATE
- net VL_SHIFT2: now also SHIFT2.-3STATE
- net VL_SHIFT3: now also SHIFT3.-3STATE
- net VL_SHIFT4: now also SHIFT4.-3STATE
Changed lines of the file:
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@@
 <net name="VCC_SHIFT1" class="0">
-<segment>
-<pinref part="SHIFT1" gate="G$1" pin="VCC"/>
-<pinref part="P+1" gate="1" pin="+5V"/>
-<wire x1="35.56" y1="63.5" x2="35.56" y2="60.96" width="0.1524" layer="91"/>
-<pinref part="SHIFT1" gate="G$1" pin="-3STATE"/>
-<wire x1="17.78" y1="50.8" x2="15.24" y2="50.8" width="0.1524" layer="91"/>
-<wire x1="15.24" y1="50.8" x2="15.24" y2="68.58" width="0.1524" layer="91"/>
-<wire x1="15.24" y1="68.58" x2="40.64" y2="68.58" width="0.1524" layer="91"/>
-<wire x1="40.64" y1="68.58" x2="40.64" y2="60.96" width="0.1524" layer="91"/>
-<wire x1="40.64" y1="60.96" x2="35.56" y2="60.96" width="0.1524" layer="91"/>
-<junction x="35.56" y="60.96"/>
-</segment>
 <segment>
 <pinref part="PWR_SHIFT1" gate="A" pin="1"/>
@@
 <pinref part="+3V1" gate="G$1" pin="+3V3"/>
 <wire x1="30.48" y1="63.5" x2="30.48" y2="60.96" width="0.1524" layer="91"/>
+<pinref part="SHIFT1" gate="G$1" pin="-3STATE"/>
+<wire x1="17.78" y1="50.8" x2="17.78" y2="60.96" width="0.1524" layer="91"/>
+<wire x1="17.78" y1="60.96" x2="30.48" y2="60.96" width="0.1524" layer="91"/>
+<junction x="30.48" y="60.96"/>
 </segment>
 <segment>
@@
 <wire x1="124.46" y1="60.96" x2="127" y2="60.96" width="0.1524" layer="91"/>
 <junction x="127" y="60.96"/>
+<pinref part="SHIFT2" gate="G$1" pin="-3STATE"/>
+<wire x1="114.3" y1="50.8" x2="114.3" y2="60.96" width="0.1524" layer="91"/>
+<wire x1="114.3" y1="60.96" x2="124.46" y2="60.96" width="0.1524" layer="91"/>
+<junction x="124.46" y="60.96"/>
 </segment>
 <segment>
@@
 </net>
 <net name="VCC_SHIFT2" class="0">
+<segment>
+<pinref part="C4" gate="G$1" pin="1"/>
+<wire x1="137.16" y1="99.06" x2="137.16" y2="104.14" width="0.1524" layer="91"/>
+<label x="134.62" y="101.6" size="1.778" layer="95" rot="R90"/>
+</segment>
+<segment>
+<pinref part="SJ1" gate="1" pin="2"/>
+<wire x1="88.9" y1="88.9" x2="96.52" y2="88.9" width="0.1524" layer="91"/>
+<label x="93.98" y="88.9" size="1.778" layer="95"/>
+</segment>
+<segment>
+<pinref part="SJ5" gate="1" pin="1"/>
+<wire x1="180.34" y1="106.68" x2="172.72" y2="106.68" width="0.1524" layer="91"/>
+<label x="160.02" y="106.68" size="1.778" layer="95"/>
+</segment>
 <segment>
 <pinref part="SHIFT2" gate="G$1" pin="VCC"/>
@@
 <wire x1="137.16" y1="60.96" x2="132.08" y2="60.96" width="0.1524" layer="91"/>
 <junction x="132.08" y="60.96"/>
-<pinref part="SHIFT2" gate="G$1" pin="-3STATE"/>
-<wire x1="114.3" y1="50.8" x2="114.3" y2="73.66" width="0.1524" layer="91"/>
-<wire x1="114.3" y1="73.66" x2="137.16" y2="73.66" width="0.1524" layer="91"/>
-<wire x1="137.16" y1="73.66" x2="137.16" y2="66.04" width="0.1524" layer="91"/>
-<junction x="137.16" y="66.04"/>
-</segment>
-<segment>
-<pinref part="C4" gate="G$1" pin="1"/>
-<wire x1="137.16" y1="99.06" x2="137.16" y2="104.14" width="0.1524" layer="91"/>
-<label x="134.62" y="101.6" size="1.778" layer="95" rot="R90"/>
-</segment>
-<segment>
-<pinref part="SJ1" gate="1" pin="2"/>
-<wire x1="88.9" y1="88.9" x2="96.52" y2="88.9" width="0.1524" layer="91"/>
-<label x="93.98" y="88.9" size="1.778" layer="95"/>
-</segment>
-<segment>
-<pinref part="SJ5" gate="1" pin="1"/>
-<wire x1="180.34" y1="106.68" x2="172.72" y2="106.68" width="0.1524" layer="91"/>
-<label x="160.02" y="106.68" size="1.778" layer="95"/>
 </segment>
 </net>
@@
 <wire x1="220.98" y1="55.88" x2="223.52" y2="55.88" width="0.1524" layer="91"/>
 <junction x="223.52" y="55.88"/>
+<pinref part="SHIFT3" gate="G$1" pin="-3STATE"/>
+<wire x1="210.82" y1="45.72" x2="210.82" y2="55.88" width="0.1524" layer="91"/>
+<wire x1="210.82" y1="55.88" x2="220.98" y2="55.88" width="0.1524" layer="91"/>
+<junction x="220.98" y="55.88"/>
 </segment>
 <segment>
@@
 <wire x1="233.68" y1="55.88" x2="228.6" y2="55.88" width="0.1524" layer="91"/>
 <junction x="228.6" y="55.88"/>
-<pinref part="SHIFT3" gate="G$1" pin="-3STATE"/>
-<wire x1="210.82" y1="45.72" x2="210.82" y2="68.58" width="0.1524" layer="91"/>
-<wire x1="210.82" y1="68.58" x2="233.68" y2="68.58" width="0.1524" layer="91"/>
-<wire x1="233.68" y1="68.58" x2="233.68" y2="60.96" width="0.1524" layer="91"/>
-<junction x="233.68" y="60.96"/>
 </segment>
 <segment>
@@
 <wire x1="320.04" y1="60.96" x2="322.58" y2="60.96" width="0.1524" layer="91"/>
 <junction x="322.58" y="60.96"/>
+<pinref part="SHIFT4" gate="G$1" pin="-3STATE"/>
+<wire x1="309.88" y1="50.8" x2="309.88" y2="60.96" width="0.1524" layer="91"/>
+<wire x1="309.88" y1="60.96" x2="320.04" y2="60.96" width="0.1524" layer="91"/>
+<junction x="320.04" y="60.96"/>
 </segment>
 <segment>
@@
 </net>
 <net name="VCC_SHIFT4" class="0">
+<segment>
+<pinref part="C8" gate="G$1" pin="1"/>
+<wire x1="335.28" y1="101.6" x2="335.28" y2="109.22" width="0.1524" layer="91"/>
+<label x="332.74" y="106.68" size="1.778" layer="95" rot="R90"/>
+</segment>
+<segment>
+<pinref part="SJ4" gate="1" pin="2"/>
+<wire x1="292.1" y1="106.68" x2="299.72" y2="106.68" width="0.1524" layer="91"/>
+<label x="297.18" y="106.68" size="1.778" layer="95"/>
+</segment>
 <segment>
 <pinref part="SHIFT4" gate="G$1" pin="VCC"/>
@@
 <wire x1="332.74" y1="60.96" x2="327.66" y2="60.96" width="0.1524" layer="91"/>
 <junction x="327.66" y="60.96"/>
-<pinref part="SHIFT4" gate="G$1" pin="-3STATE"/>
-<wire x1="309.88" y1="50.8" x2="309.88" y2="73.66" width="0.1524" layer="91"/>
-<wire x1="309.88" y1="73.66" x2="332.74" y2="73.66" width="0.1524" layer="91"/>
-<wire x1="332.74" y1="73.66" x2="332.74" y2="66.04" width="0.1524" layer="91"/>
-<junction x="332.74" y="66.04"/>
-</segment>
-<segment>
-<pinref part="C8" gate="G$1" pin="1"/>
-<wire x1="335.28" y1="101.6" x2="335.28" y2="109.22" width="0.1524" layer="91"/>
-<label x="332.74" y="106.68" size="1.778" layer="95" rot="R90"/>
-</segment>
-<segment>
-<pinref part="SJ4" gate="1" pin="2"/>
-<wire x1="292.1" y1="106.68" x2="299.72" y2="106.68" width="0.1524" layer="91"/>
-<label x="297.18" y="106.68" size="1.778" layer="95"/>
-</segment>
-</net>
+</segment>
+</net>
+<net name="+5V" class="0">
+<segment>
+<pinref part="SHIFT1" gate="G$1" pin="VCC"/>
+<pinref part="P+1" gate="1" pin="+5V"/>
+<wire x1="35.56" y1="63.5" x2="35.56" y2="60.96" width="0.1524" layer="91"/>
+</segment>
+</net>
