File: max33xxE_breakout.brd (EAGLE design)
At the start: 48.3 x 15.2 mm, 30 parts

Commit message: forgot that the -THREESTATE *must* be pulled to VCC/VL
Connections:
- net VCC_SHIFT1: now also SHIFT1.8
- net VCC_SHIFT2: now also SHIFT2.8
- net VCC_SHIFT3: now also SHIFT3.8
- net VCC_SHIFT4: now also SHIFT4.8
Routing:
- net VCC_SHIFT4: track 6.09 -> 12.7 mm
- net VCC_SHIFT1: track 11.7 -> 13.0 mm
- net VCC_SHIFT3: track 14.0 -> 15.4 mm
- net VCC_SHIFT2: track 13.6 -> 15.0 mm
Changed lines of the file:
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@@
 <setting verticaltext="up"/>
 </settings>
-<grid distance="12.5" unitdist="mil" unit="mil" style="lines" multiple="1" display="yes" altdistance="0.025" altunitdist="inch" altunit="inch"/>
+<grid distance="1" unitdist="mil" unit="mil" style="lines" multiple="1" display="yes" altdistance="0.025" altunitdist="inch" altunit="inch"/>
 <layers>
 <layer number="1" name="Top" color="4" fill="1" visible="yes" active="yes"/>
@@
 <wire x1="10.922" y1="10.16" x2="10.63625" y2="10.16" width="0.254" layer="1"/>
 <wire x1="10.63625" y1="10.16" x2="9.68375" y2="9.2075" width="0.254" layer="1"/>
-<wire x1="9.68375" y1="9.2075" x2="5.0546" y2="9.2075" width="0.254" layer="1"/>
+<wire x1="9.68375" y1="9.2075" x2="8.9662" y2="9.2075" width="0.254" layer="1"/>
+<wire x1="8.9662" y1="9.2075" x2="5.0546" y2="9.2075" width="0.254" layer="1"/>
 <wire x1="5.0546" y1="9.2075" x2="5.0546" y2="10.4928" width="0.254" layer="1"/>
 <wire x1="5.0546" y1="10.4928" x2="5.035" y2="10.5378" width="0.254" layer="1"/>
+<contactref element="SHIFT1" pad="8"/>
+<wire x1="8.935" y1="10.5378" x2="8.9662" y2="10.5378" width="0.254" layer="1"/>
+<wire x1="8.9662" y1="10.5378" x2="8.9662" y2="9.2075" width="0.254" layer="1"/>
 </signal>
 <signal name="VL_SHIFT1">
@@
 <wire x1="23.622" y1="10.16" x2="23.33625" y2="10.16" width="0.254" layer="1"/>
 <wire x1="23.33625" y1="10.16" x2="22.38375" y2="9.2075" width="0.254" layer="1"/>
-<wire x1="22.38375" y1="9.2075" x2="17.7546" y2="9.2075" width="0.254" layer="1"/>
+<wire x1="22.38375" y1="9.2075" x2="21.6662" y2="9.2075" width="0.254" layer="1"/>
+<wire x1="21.6662" y1="9.2075" x2="17.7546" y2="9.2075" width="0.254" layer="1"/>
 <wire x1="17.7546" y1="9.2075" x2="17.7546" y2="10.4674" width="0.254" layer="1"/>
 <wire x1="17.7546" y1="10.4674" x2="17.735" y2="10.5378" width="0.254" layer="1"/>
+<contactref element="SHIFT2" pad="8"/>
+<wire x1="21.635" y1="10.5378" x2="21.6662" y2="10.5378" width="0.254" layer="1"/>
+<wire x1="21.6662" y1="10.5378" x2="21.6662" y2="9.2075" width="0.254" layer="1"/>
 </signal>
 <signal name="IOVCC4_SHIFT3">
@@
 <wire x1="36.322" y1="10.16" x2="36.03625" y2="10.16" width="0.254" layer="1"/>
 <wire x1="36.03625" y1="10.16" x2="35.08375" y2="9.2075" width="0.254" layer="1"/>
-<wire x1="35.08375" y1="9.2075" x2="30.4546" y2="9.2075" width="0.254" layer="1"/>
+<wire x1="35.08375" y1="9.2075" x2="34.3662" y2="9.2075" width="0.254" layer="1"/>
+<wire x1="34.3662" y1="9.2075" x2="30.4546" y2="9.2075" width="0.254" layer="1"/>
 <wire x1="30.4546" y1="9.2075" x2="30.4546" y2="10.5182" width="0.254" layer="1"/>
 <wire x1="30.4546" y1="10.5182" x2="30.435" y2="10.5378" width="0.254" layer="1"/>
+<contactref element="SHIFT3" pad="8"/>
+<wire x1="34.335" y1="10.5378" x2="34.3662" y2="10.5378" width="0.254" layer="1"/>
+<wire x1="34.3662" y1="10.5378" x2="34.3662" y2="9.2075" width="0.254" layer="1"/>
 </signal>
 <signal name="IOVCC4_SHIFT4">
@@
 <wire x1="39.4716" y1="10.2108" x2="39.37" y2="10.16" width="0.254" layer="1"/>
 <wire x1="39.37" y1="10.16" x2="37.338" y2="10.16" width="0.254" layer="1"/>
+<contactref element="SHIFT4" pad="8"/>
+<wire x1="43.135" y1="10.5378" x2="43.1546" y2="10.5886" width="0.254" layer="1"/>
+<wire x1="43.1546" y1="10.5886" x2="43.1546" y2="9.2075" width="0.254" layer="1"/>
+<wire x1="43.1546" y1="9.2075" x2="46.99" y2="9.2075" width="0.254" layer="1"/>
+<wire x1="46.99" y1="9.2075" x2="47.035" y2="9.2075" width="0.254" layer="1"/>
+<wire x1="47.035" y1="9.2075" x2="47.035" y2="10.5378" width="0.254" layer="1"/>
 </signal>
 </signals>

Commit message: daym, -threestate must be pulled VL not VCC, good that I verified this...
Connections:
- new net +5V: SHIFT1.14
- net VCC_SHIFT1: no longer SHIFT1.14, SHIFT1.8
- net VCC_SHIFT2: no longer SHIFT2.8
- net VCC_SHIFT3: no longer SHIFT3.8
- net VCC_SHIFT4: no longer SHIFT4.8
- net VL_SHIFT1: now also SHIFT1.8
- net VL_SHIFT2: now also SHIFT2.8
- net VL_SHIFT3: now also SHIFT3.8
- net VL_SHIFT4: now also SHIFT4.8
Routing:
- net VCC_SHIFT4: track 12.7 -> 6.10 mm
- net VCC_SHIFT2: track 15.0 -> 13.5 mm
- net VCC_SHIFT1: track 13.0 -> 11.6 mm
- net VCC_SHIFT3: track 15.4 -> 14.0 mm
Changed lines of the file:
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@@
 </signal>
 <signal name="VCC_SHIFT1">
-<contactref element="SHIFT1" pad="14"/>
 <contactref element="PWR_SHIFT1" pad="1"/>
 <contactref element="C2" pad="1"/>
 <contactref element="SJ1" pad="1"/>
 <wire x1="3.5052" y1="10.5156" x2="5.0292" y2="10.5156" width="0.254" layer="1"/>
-<wire x1="5.0292" y1="10.5156" x2="5.035" y2="10.5378" width="0.254" layer="1"/>
 <wire x1="3.5052" y1="10.5156" x2="3.4925" y2="10.4" width="0.254" layer="1"/>
 <wire x1="1.3716" y1="10.3632" x2="3.3528" y2="10.3632" width="0.254" layer="1"/>
@@
 <wire x1="8.9662" y1="9.2075" x2="5.0546" y2="9.2075" width="0.254" layer="1"/>
 <wire x1="5.0546" y1="9.2075" x2="5.0546" y2="10.4928" width="0.254" layer="1"/>
-<wire x1="5.0546" y1="10.4928" x2="5.035" y2="10.5378" width="0.254" layer="1"/>
-<contactref element="SHIFT1" pad="8"/>
-<wire x1="8.935" y1="10.5378" x2="8.9662" y2="10.5378" width="0.254" layer="1"/>
-<wire x1="8.9662" y1="10.5378" x2="8.9662" y2="9.2075" width="0.254" layer="1"/>
+<wire x1="5.0546" y1="10.4928" x2="5.0292" y2="10.5156" width="0" layer="19" extent="1-1"/>
 </signal>
 <signal name="VL_SHIFT1">
@@
 <wire x1="10.4775" y1="5.08" x2="1.27" y2="5.08" width="0.254" layer="16"/>
 <wire x1="10.4775" y1="5.08" x2="10.922" y2="5.08" width="0.254" layer="1"/>
+<contactref element="SHIFT1" pad="8"/>
+<wire x1="10.4775" y1="5.08" x2="8.935" y2="10.5378" width="0" layer="19" extent="1-1"/>
 </signal>
 <signal name="IOVL2_SHIFT1">
@@
 <wire x1="23.1775" y1="5.08" x2="13.97" y2="5.08" width="0.254" layer="16"/>
 <wire x1="23.1775" y1="5.08" x2="23.622" y2="5.08" width="0.254" layer="1"/>
+<contactref element="SHIFT2" pad="8"/>
+<wire x1="23.1775" y1="5.08" x2="21.635" y2="10.5378" width="0" layer="19" extent="1-1"/>
 </signal>
 <signal name="VCC_SHIFT2">
-<contactref element="SHIFT2" pad="14"/>
-<contactref element="PWR_SHIFT2" pad="1"/>
 <contactref element="C4" pad="1"/>
 <contactref element="SJ1" pad="2"/>
 <contactref element="SJ5" pad="1"/>
 <wire x1="16.3068" y1="10.5156" x2="17.6784" y2="10.5156" width="0.254" layer="1"/>
-<wire x1="17.6784" y1="10.5156" x2="17.735" y2="10.5378" width="0.254" layer="1"/>
 <wire x1="16.3068" y1="10.5156" x2="16.1925" y2="10.4" width="0.254" layer="1"/>
 <wire x1="14.0208" y1="10.3632" x2="16.1544" y2="10.3632" width="0.254" layer="1"/>
 <wire x1="14.0208" y1="10.2108" x2="14.0208" y2="10.3632" width="0.254" layer="1"/>
 <wire x1="16.1544" y1="10.3632" x2="16.1925" y2="10.4" width="0.254" layer="1"/>
-<wire x1="14.0208" y1="10.2108" x2="13.97" y2="10.16" width="0.254" layer="1"/>
-<wire x1="13.97" y1="10.16" x2="11.938" y2="10.16" width="0.254" layer="1"/>
 <wire x1="23.622" y1="10.16" x2="23.33625" y2="10.16" width="0.254" layer="1"/>
 <wire x1="23.33625" y1="10.16" x2="22.38375" y2="9.2075" width="0.254" layer="1"/>
@@
 <wire x1="21.6662" y1="9.2075" x2="17.7546" y2="9.2075" width="0.254" layer="1"/>
 <wire x1="17.7546" y1="9.2075" x2="17.7546" y2="10.4674" width="0.254" layer="1"/>
-<wire x1="17.7546" y1="10.4674" x2="17.735" y2="10.5378" width="0.254" layer="1"/>
-<contactref element="SHIFT2" pad="8"/>
-<wire x1="21.635" y1="10.5378" x2="21.6662" y2="10.5378" width="0.254" layer="1"/>
-<wire x1="21.6662" y1="10.5378" x2="21.6662" y2="9.2075" width="0.254" layer="1"/>
+<wire x1="11.938" y1="10.16" x2="14.0208" y2="10.16" width="0.254" layer="1"/>
+<wire x1="14.0208" y1="10.16" x2="14.0208" y2="10.2108" width="0.254" layer="1"/>
+<contactref element="SHIFT2" pad="14"/>
+<contactref element="PWR_SHIFT2" pad="1"/>
+<wire x1="17.7546" y1="10.4674" x2="17.735" y2="10.5378" width="0" layer="19" extent="1-1"/>
+<wire x1="17.6784" y1="10.5156" x2="17.735" y2="10.5378" width="0" layer="19" extent="1-1"/>
+<wire x1="13.97" y1="10.16" x2="14.0208" y2="10.16" width="0" layer="19" extent="1-1"/>
 </signal>
 <signal name="IOVCC4_SHIFT3">
@@
 <wire x1="35.8775" y1="5.08" x2="26.67" y2="5.08" width="0.254" layer="16"/>
 <wire x1="35.8775" y1="5.08" x2="36.322" y2="5.08" width="0.254" layer="1"/>
+<contactref element="SHIFT3" pad="8"/>
+<wire x1="35.8775" y1="5.08" x2="34.335" y2="10.5378" width="0" layer="19" extent="1-1"/>
 </signal>
 <signal name="VCC_SHIFT3">
@@
 <wire x1="30.4546" y1="9.2075" x2="30.4546" y2="10.5182" width="0.254" layer="1"/>
 <wire x1="30.4546" y1="10.5182" x2="30.435" y2="10.5378" width="0.254" layer="1"/>
-<contactref element="SHIFT3" pad="8"/>
-<wire x1="34.335" y1="10.5378" x2="34.3662" y2="10.5378" width="0.254" layer="1"/>
-<wire x1="34.3662" y1="10.5378" x2="34.3662" y2="9.2075" width="0.254" layer="1"/>
 </signal>
 <signal name="IOVCC4_SHIFT4">
@@
 <wire x1="39.4716" y1="5.0292" x2="39.37" y2="5.08" width="0.254" layer="1"/>
 <wire x1="39.37" y1="5.08" x2="37.338" y2="5.08" width="0.254" layer="1"/>
+<contactref element="SHIFT4" pad="8"/>
+<wire x1="43.1292" y1="4.7244" x2="47.035" y2="10.5378" width="0" layer="19" extent="1-1"/>
 </signal>
 <signal name="VCC_SHIFT4">
-<contactref element="SHIFT4" pad="14"/>
-<contactref element="PWR_SHIFT4" pad="1"/>
 <contactref element="C8" pad="1"/>
 <contactref element="SJ4" pad="2"/>
 <wire x1="41.6052" y1="10.5156" x2="43.1292" y2="10.5156" width="0.254" layer="1"/>
-<wire x1="43.1292" y1="10.5156" x2="43.135" y2="10.5378" width="0.254" layer="1"/>
 <wire x1="41.6052" y1="10.5156" x2="41.5925" y2="10.4" width="0.254" layer="1"/>
 <wire x1="39.4716" y1="10.3632" x2="41.4528" y2="10.3632" width="0.254" layer="1"/>
 <wire x1="39.4716" y1="10.2108" x2="39.4716" y2="10.3632" width="0.254" layer="1"/>
 <wire x1="41.4528" y1="10.3632" x2="41.5925" y2="10.4" width="0.254" layer="1"/>
-<wire x1="39.4716" y1="10.2108" x2="39.37" y2="10.16" width="0.254" layer="1"/>
-<wire x1="39.37" y1="10.16" x2="37.338" y2="10.16" width="0.254" layer="1"/>
-<contactref element="SHIFT4" pad="8"/>
-<wire x1="43.135" y1="10.5378" x2="43.1546" y2="10.5886" width="0.254" layer="1"/>
-<wire x1="43.1546" y1="10.5886" x2="43.1546" y2="9.2075" width="0.254" layer="1"/>
-<wire x1="43.1546" y1="9.2075" x2="46.99" y2="9.2075" width="0.254" layer="1"/>
-<wire x1="46.99" y1="9.2075" x2="47.035" y2="9.2075" width="0.254" layer="1"/>
-<wire x1="47.035" y1="9.2075" x2="47.035" y2="10.5378" width="0.254" layer="1"/>
+<wire x1="37.338" y1="10.16" x2="39.4716" y2="10.16" width="0.254" layer="1"/>
+<wire x1="39.4716" y1="10.16" x2="39.4716" y2="10.2108" width="0.254" layer="1"/>
+<contactref element="SHIFT4" pad="14"/>
+<contactref element="PWR_SHIFT4" pad="1"/>
+<wire x1="43.1292" y1="10.5156" x2="43.135" y2="10.5378" width="0" layer="19" extent="1-1"/>
+<wire x1="39.37" y1="10.16" x2="39.4716" y2="10.16" width="0" layer="19" extent="1-1"/>
+</signal>
+<signal name="+5V">
+<contactref element="SHIFT1" pad="14"/>
 </signal>
 </signals>

Commit message: route the VL pull-ups via bottom
Routing:
- net VL_SHIFT4: track 6.09 -> 20.3 mm, vias 0 -> 2
- net VL_SHIFT2: track 15.7 -> 24.3 mm, vias 1 -> 2
- net VL_SHIFT3: track 15.7 -> 24.2 mm, vias 1 -> 2
- net VL_SHIFT1: track 13.7 -> 22.2 mm, vias 1 -> 2
Changed lines of the file:
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@@
 <setting verticaltext="up"/>
 </settings>
-<grid distance="1" unitdist="mil" unit="mil" style="lines" multiple="1" display="yes" altdistance="0.025" altunitdist="inch" altunit="inch"/>
+<grid distance="6.25" unitdist="mil" unit="mil" style="lines" multiple="1" display="yes" altdistance="0.025" altunitdist="inch" altunit="inch"/>
 <layers>
 <layer number="1" name="Top" color="4" fill="1" visible="yes" active="yes"/>
@@
 <wire x1="10.4775" y1="5.08" x2="10.922" y2="5.08" width="0.254" layer="1"/>
 <contactref element="SHIFT1" pad="8"/>
-<wire x1="10.4775" y1="5.08" x2="8.935" y2="10.5378" width="0" layer="19" extent="1-1"/>
+<via x="9.2075" y="11.27125" extent="1-16" drill="0.6096"/>
+<wire x1="10.4775" y1="5.08" x2="9.2075" y2="5.08" width="0.254" layer="16"/>
+<wire x1="9.2075" y1="5.08" x2="9.2075" y2="11.27125" width="0.254" layer="16"/>
+<wire x1="9.2075" y1="11.27125" x2="8.935" y2="11.27125" width="0.254" layer="1"/>
+<wire x1="8.935" y1="11.27125" x2="8.935" y2="10.5378" width="0.254" layer="1"/>
 </signal>
 <signal name="IOVL2_SHIFT1">
@@
 <wire x1="23.1775" y1="5.08" x2="23.622" y2="5.08" width="0.254" layer="1"/>
 <contactref element="SHIFT2" pad="8"/>
-<wire x1="23.1775" y1="5.08" x2="21.635" y2="10.5378" width="0" layer="19" extent="1-1"/>
+<via x="21.83765" y="11.32205" extent="1-16" drill="0.6096"/>
+<wire x1="23.1775" y1="5.08" x2="21.83765" y2="5.08" width="0.254" layer="16"/>
+<wire x1="21.83765" y1="5.08" x2="21.83765" y2="11.32205" width="0.254" layer="16"/>
+<wire x1="21.83765" y1="11.32205" x2="21.635" y2="11.32205" width="0.254" layer="1"/>
+<wire x1="21.635" y1="11.32205" x2="21.635" y2="10.5378" width="0.254" layer="1"/>
 </signal>
 <signal name="VCC_SHIFT2">
@@
 <wire x1="35.8775" y1="5.08" x2="36.322" y2="5.08" width="0.254" layer="1"/>
 <contactref element="SHIFT3" pad="8"/>
-<wire x1="35.8775" y1="5.08" x2="34.335" y2="10.5378" width="0" layer="19" extent="1-1"/>
+<via x="34.6075" y="11.27125" extent="1-16" drill="0.6096"/>
+<wire x1="35.8775" y1="5.08" x2="34.6075" y2="5.08" width="0.254" layer="16"/>
+<wire x1="34.6075" y1="5.08" x2="34.6075" y2="11.27125" width="0.254" layer="16"/>
+<wire x1="34.6075" y1="11.27125" x2="34.335" y2="11.27125" width="0.254" layer="1"/>
+<wire x1="34.335" y1="11.27125" x2="34.335" y2="10.5378" width="0.254" layer="1"/>
 </signal>
 <signal name="VCC_SHIFT3">
@@
 <wire x1="39.37" y1="5.08" x2="37.338" y2="5.08" width="0.254" layer="1"/>
 <contactref element="SHIFT4" pad="8"/>
-<wire x1="43.1292" y1="4.7244" x2="47.035" y2="10.5378" width="0" layer="19" extent="1-1"/>
+<via x="41.5925" y="4.28625" extent="1-16" drill="0.6096"/>
+<via x="47.3075" y="11.27125" extent="1-16" drill="0.6096"/>
+<wire x1="47.3075" y1="11.27125" x2="47.3075" y2="4.28625" width="0.254" layer="16"/>
+<wire x1="47.3075" y1="4.28625" x2="41.5925" y2="4.28625" width="0.254" layer="16"/>
+<wire x1="47.3075" y1="11.27125" x2="47.035" y2="11.27125" width="0.254" layer="1"/>
+<wire x1="47.035" y1="11.27125" x2="47.035" y2="10.5378" width="0.254" layer="1"/>
+<wire x1="41.5925" y1="4.28625" x2="41.5925" y2="4.84" width="0.254" layer="1"/>
 </signal>
 <signal name="VCC_SHIFT4">
